Commit message: add gripper in URDF

File: foodly_rd_description/urdf/foodly_rd_left_gripper.xacro (robot description, xacro)
@@ -4,14 +4,14 @@
     <link name="${NAME_LINK_ARM_L_7}">
       <visual>
-        <origin rpy="0 0 0" xyz="0.0 0.0 0.0"/>
+        <origin rpy="0 0 0" xyz="-0.035 -0.000 -1.012"/>
         <geometry>
-          <mesh filename="${VISUAL_MESH_PATH}/L_Link7.stl" scale="1.0 1.0 1.0"/>
+          <mesh filename="${VISUAL_MESH_PATH}/Gripper_v23.2.STL" scale="0.001 0.001 0.001"/>
         </geometry>
         <material name="${COLOR_LINK_GRIPPER}"/>
       </visual>
       <collision>
-        <origin rpy="0 0 0" xyz="0.0 0.0 0.0"/>
+        <origin rpy="0 0 0" xyz="-0.035 -0.000 -1.012"/>
         <geometry>
-          <mesh filename="${COLLISION_MESH_PATH}/L_Link7.stl" scale="1.0 1.0 1.0"/>
+          <mesh filename="${COLLISION_MESH_PATH}/Gripper_v23.2.STL" scale="0.001 0.001 0.001"/>
         </geometry>
       </collision>
@@ -37,5 +37,5 @@
         <origin rpy="0 0 0" xyz="0.0 0.0 0.0"/>
         <geometry>
-          <mesh filename="${VISUAL_MESH_PATH}/L_GripperA.stl" scale="1.0 1.0 1.0"/>
+          <mesh filename="${VISUAL_MESH_PATH}/L_GripperA.stl" scale="0.01 0.01 0.01"/>
         </geometry>
         <material name="${COLOR_LINK_GRIPPER}"/>
@@ -44,5 +44,5 @@
         <origin rpy="0 0 0" xyz="0.0 0.0 0.0"/>
         <geometry>
-          <mesh filename="${COLLISION_MESH_PATH}/L_GripperA.stl" scale="1.0 1.0 1.0"/>
+          <mesh filename="${COLLISION_MESH_PATH}/L_GripperA.stl" scale="0.01 0.01 0.01"/>
         </geometry>
       </collision>
@@ -57,5 +57,5 @@
         <origin rpy="0 0 0" xyz="0.0 0.0 0.0"/>
         <geometry>
-            <mesh filename="${VISUAL_MESH_PATH}/Tong.stl" />
+            <mesh filename="${VISUAL_MESH_PATH}/Tong.stl" scale="0.01 0.01 0.01" />
         </geometry>
         <material name="${COLOR_LINK_GRIPPER}"/>
@@ -64,5 +64,5 @@
         <origin rpy="0 0 0" xyz="0.0 0.0 0.0"/>
         <geometry>
-          <mesh filename="${COLLISION_MESH_PATH}/Tong.stl" />
+          <mesh filename="${COLLISION_MESH_PATH}/Tong.stl" scale="0.01 0.01 0.01" />
         </geometry>
       </collision>
@@ -97,5 +97,5 @@
         <origin rpy="0 0 0" xyz="0.0 0.0 0.0"/>
         <geometry>
-          <mesh filename="${VISUAL_MESH_PATH}/L_GripperB.stl" scale="1.0 1.0 1.0"/>
+          <mesh filename="${VISUAL_MESH_PATH}/L_GripperB.stl" scale="0.01 0.01 0.01"/>
         </geometry>
         <material name="${COLOR_LINK_GRIPPER}"/>
@@ -104,5 +104,5 @@
         <origin rpy="0 0 0" xyz="0.0 0.0 0.0"/>
         <geometry>
-          <mesh filename="${COLLISION_MESH_PATH}/L_GripperB.stl" scale="1.0 1.0 1.0"/>
+          <mesh filename="${COLLISION_MESH_PATH}/L_GripperB.stl" scale="0.01 0.01 0.01"/>
         </geometry>
       </collision>
@@ -117,5 +117,5 @@
         <origin rpy="0 0 3.1415" xyz="0.0 0.0 0.0"/>
         <geometry>
-            <mesh filename="${VISUAL_MESH_PATH}/Tong.stl" />
+            <mesh filename="${VISUAL_MESH_PATH}/Tong.stl" scale="0.01 0.01 0.01" />
         </geometry>
         <material name="${COLOR_LINK_GRIPPER}"/>
@@ -124,5 +124,5 @@
         <origin rpy="0 0 3.1415" xyz="0.0 0.0 0.0"/>
         <geometry>
-          <mesh filename="${COLLISION_MESH_PATH}/Tong.stl" />
+          <mesh filename="${COLLISION_MESH_PATH}/Tong.stl" scale="0.01 0.01 0.01" />
         </geometry>
       </collision>

File: foodly_rd_description/urdf/foodly_rd_right_gripper.xacro (robot description, xacro)
@@ -4,14 +4,14 @@
     <link name="${NAME_LINK_ARM_R_7}">
       <visual>
-        <origin rpy="0 0 0" xyz="0.0 0.0 0.0"/>
+        <origin rpy="0 0 3.14" xyz="0.035 0.0 -1.012"/>
         <geometry>
-          <mesh filename="${VISUAL_MESH_PATH}/R_Link7.stl" scale="1.0 1.0 1.0"/>
+          <mesh filename="${VISUAL_MESH_PATH}/Gripper_v23.2.STL" scale="0.001 0.001 0.001"/>
         </geometry>
         <material name="${COLOR_LINK_GRIPPER}"/>
       </visual>
       <collision>
-        <origin rpy="0 0 0" xyz="0.0 0.0 0.0"/>
+        <origin rpy="0 0 3.14" xyz="0.01 0.0 -1.012"/>
         <geometry>
-          <mesh filename="${COLLISION_MESH_PATH}/R_Link7.stl" scale="1.0 1.0 1.0"/>
+          <mesh filename="${COLLISION_MESH_PATH}/Gripper_v23.2.STL" scale="0.001 0.001 0.001"/>
         </geometry>
       </collision>
@@ -37,5 +37,5 @@
         <origin rpy="0 0 0" xyz="0.0 0.0 0.0"/>
         <geometry>
-          <mesh filename="${VISUAL_MESH_PATH}/R_GripperA.stl" scale="1.0 1.0 1.0"/>
+          <mesh filename="${VISUAL_MESH_PATH}/R_GripperA.stl" scale="0.001 0.001 0.001"/>
         </geometry>
         <material name="${COLOR_LINK_GRIPPER}"/>
@@ -44,5 +44,5 @@
         <origin rpy="0 0 0" xyz="0.0 0.0 0.0"/>
         <geometry>
-          <mesh filename="${COLLISION_MESH_PATH}/R_GripperA.stl" scale="1.0 1.0 1.0"/>
+          <mesh filename="${COLLISION_MESH_PATH}/R_GripperA.stl" scale="0.001 0.001 0.001"/>
         </geometry>
       </collision>
@@ -57,5 +57,5 @@
         <origin rpy="0 0 3.14" xyz="0.0 0.0 0.0"/>
         <geometry>
-            <mesh filename="${VISUAL_MESH_PATH}/Tong.stl" />
+            <mesh filename="${VISUAL_MESH_PATH}/Tong.stl" scale="0.001 0.001 0.001"/>
         </geometry>
         <material name="${COLOR_LINK_GRIPPER}"/>
@@ -64,5 +64,5 @@
         <origin rpy="0 0 3.14" xyz="0.0 0.0 0.0"/>
         <geometry>
-          <mesh filename="${COLLISION_MESH_PATH}/Tong.stl" />
+          <mesh filename="${COLLISION_MESH_PATH}/Tong.stl" scale="0.001 0.001 0.001"/>
         </geometry>
       </collision>
@@ -97,5 +97,5 @@
         <origin rpy="0 0 0" xyz="0.0 0.0 0.0"/>
         <geometry>
-          <mesh filename="${VISUAL_MESH_PATH}/R_GripperB.stl" scale="1.0 1.0 1.0"/>
+          <mesh filename="${VISUAL_MESH_PATH}/R_GripperB.stl" scale="0.001 0.001 0.001"/>
         </geometry>
         <material name="${COLOR_LINK_GRIPPER}"/>
@@ -104,5 +104,5 @@
         <origin rpy="0 0 0" xyz="0.0 0.0 0.0"/>
         <geometry>
-          <mesh filename="${COLLISION_MESH_PATH}/R_GripperB.stl" scale="1.0 1.0 1.0"/>
+          <mesh filename="${COLLISION_MESH_PATH}/R_GripperB.stl" scale="0.001 0.001 0.001"/>
         </geometry>
       </collision>
@@ -117,5 +117,5 @@
         <origin rpy="0 0 0" xyz="0.0 0.0 0.0"/>
         <geometry>
-            <mesh filename="${VISUAL_MESH_PATH}/Tong.stl" />
+            <mesh filename="${VISUAL_MESH_PATH}/Tong.stl" scale="0.001 0.001 0.001"/>
         </geometry>
         <material name="${COLOR_LINK_GRIPPER}"/>
@@ -124,5 +124,5 @@
         <origin rpy="0 0 0" xyz="0.0 0.0 0.0"/>
         <geometry>
-          <mesh filename="${COLLISION_MESH_PATH}/Tong.stl" />
+          <mesh filename="${COLLISION_MESH_PATH}/Tong.stl" scale="0.001 0.001 0.001"/>
         </geometry>
       </collision>

Commit message: update urdf

File: foodly_rd_description/urdf/foodly_rd_left_gripper.xacro (robot description, xacro)
@@ -4,5 +4,5 @@
     <link name="${NAME_LINK_ARM_L_7}">
       <visual>
-        <origin rpy="0 0 0" xyz="-0.035 -0.000 -1.012"/>
+        <origin rpy="0 0 0" xyz="-0.035 0.0 -1.012"/>
         <geometry>
           <mesh filename="${VISUAL_MESH_PATH}/Gripper_v23.2.STL" scale="0.001 0.001 0.001"/>
@@ -11,5 +11,5 @@
       </visual>
       <collision>
-        <origin rpy="0 0 0" xyz="-0.035 -0.000 -1.012"/>
+        <origin rpy="0 0 0" xyz="-0.035 0.0 -1.012"/>
         <geometry>
           <mesh filename="${COLLISION_MESH_PATH}/Gripper_v23.2.STL" scale="0.001 0.001 0.001"/>

File: foodly_rd_description/urdf/foodly_rd_right_gripper.xacro (robot description, xacro)
@@ -11,5 +11,5 @@
       </visual>
       <collision>
-        <origin rpy="0 0 3.14" xyz="0.01 0.0 -1.012"/>
+        <origin rpy="0 0 3.14" xyz="0.035 0.0 -1.012"/>
         <geometry>
           <mesh filename="${COLLISION_MESH_PATH}/Gripper_v23.2.STL" scale="0.001 0.001 0.001"/>

Commit message: update error state machine

File: foodly_rd_description/urdf/foodly_rd_left_gripper.xacro (robot description, xacro)
@@ -4,14 +4,14 @@
     <link name="${NAME_LINK_ARM_L_7}">
       <visual>
-        <origin rpy="0 0 0" xyz="-0.035 0.0 -1.012"/>
+        <origin rpy="0 0 0" xyz="0.0 0.0 0.0"/>
         <geometry>
-          <mesh filename="${VISUAL_MESH_PATH}/Gripper_v23.2.STL" scale="0.001 0.001 0.001"/>
+          <mesh filename="${VISUAL_MESH_PATH}/L_Link7.stl" scale="1.0 1.0 1.0"/>
         </geometry>
         <material name="${COLOR_LINK_GRIPPER}"/>
       </visual>
       <collision>
-        <origin rpy="0 0 0" xyz="-0.035 0.0 -1.012"/>
+        <origin rpy="0 0 0" xyz="0.0 0.0 0.0"/>
         <geometry>
-          <mesh filename="${COLLISION_MESH_PATH}/Gripper_v23.2.STL" scale="0.001 0.001 0.001"/>
+          <mesh filename="${COLLISION_MESH_PATH}/L_Link7.stl" scale="1.0 1.0 1.0"/>
         </geometry>
       </collision>
@@ -37,5 +37,5 @@
         <origin rpy="0 0 0" xyz="0.0 0.0 0.0"/>
         <geometry>
-          <mesh filename="${VISUAL_MESH_PATH}/L_GripperA.stl" scale="0.01 0.01 0.01"/>
+          <mesh filename="${VISUAL_MESH_PATH}/L_GripperA.stl" scale="1.0 1.0 1.0"/>
         </geometry>
         <material name="${COLOR_LINK_GRIPPER}"/>
@@ -44,5 +44,5 @@
         <origin rpy="0 0 0" xyz="0.0 0.0 0.0"/>
         <geometry>
-          <mesh filename="${COLLISION_MESH_PATH}/L_GripperA.stl" scale="0.01 0.01 0.01"/>
+          <mesh filename="${COLLISION_MESH_PATH}/L_GripperA.stl" scale="1.0 1.0 1.0"/>
         </geometry>
       </collision>
@@ -57,5 +57,5 @@
         <origin rpy="0 0 0" xyz="0.0 0.0 0.0"/>
         <geometry>
-            <mesh filename="${VISUAL_MESH_PATH}/Tong.stl" scale="0.01 0.01 0.01" />
+            <mesh filename="${VISUAL_MESH_PATH}/Tong.stl" />
         </geometry>
         <material name="${COLOR_LINK_GRIPPER}"/>
@@ -64,5 +64,5 @@
         <origin rpy="0 0 0" xyz="0.0 0.0 0.0"/>
         <geometry>
-          <mesh filename="${COLLISION_MESH_PATH}/Tong.stl" scale="0.01 0.01 0.01" />
+          <mesh filename="${COLLISION_MESH_PATH}/Tong.stl" />
         </geometry>
       </collision>
@@ -97,5 +97,5 @@
         <origin rpy="0 0 0" xyz="0.0 0.0 0.0"/>
         <geometry>
-          <mesh filename="${VISUAL_MESH_PATH}/L_GripperB.stl" scale="0.01 0.01 0.01"/>
+          <mesh filename="${VISUAL_MESH_PATH}/L_GripperB.stl" scale="1.0 1.0 1.0"/>
         </geometry>
         <material name="${COLOR_LINK_GRIPPER}"/>
@@ -104,5 +104,5 @@
         <origin rpy="0 0 0" xyz="0.0 0.0 0.0"/>
         <geometry>
-          <mesh filename="${COLLISION_MESH_PATH}/L_GripperB.stl" scale="0.01 0.01 0.01"/>
+          <mesh filename="${COLLISION_MESH_PATH}/L_GripperB.stl" scale="1.0 1.0 1.0"/>
         </geometry>
       </collision>
@@ -117,5 +117,5 @@
         <origin rpy="0 0 3.1415" xyz="0.0 0.0 0.0"/>
         <geometry>
-            <mesh filename="${VISUAL_MESH_PATH}/Tong.stl" scale="0.01 0.01 0.01" />
+            <mesh filename="${VISUAL_MESH_PATH}/Tong.stl" />
         </geometry>
         <material name="${COLOR_LINK_GRIPPER}"/>
@@ -124,5 +124,5 @@
         <origin rpy="0 0 3.1415" xyz="0.0 0.0 0.0"/>
         <geometry>
-          <mesh filename="${COLLISION_MESH_PATH}/Tong.stl" scale="0.01 0.01 0.01" />
+          <mesh filename="${COLLISION_MESH_PATH}/Tong.stl" />
         </geometry>
       </collision>

File: foodly_rd_description/urdf/foodly_rd_right_gripper.xacro (robot description, xacro)
@@ -4,14 +4,14 @@
     <link name="${NAME_LINK_ARM_R_7}">
       <visual>
-        <origin rpy="0 0 3.14" xyz="0.035 0.0 -1.012"/>
+        <origin rpy="0 0 0" xyz="0.0 0.0 0.0"/>
         <geometry>
-          <mesh filename="${VISUAL_MESH_PATH}/Gripper_v23.2.STL" scale="0.001 0.001 0.001"/>
+          <mesh filename="${VISUAL_MESH_PATH}/R_Link7.stl" scale="1.0 1.0 1.0"/>
         </geometry>
         <material name="${COLOR_LINK_GRIPPER}"/>
       </visual>
       <collision>
-        <origin rpy="0 0 3.14" xyz="0.035 0.0 -1.012"/>
+        <origin rpy="0 0 0" xyz="0.0 0.0 0.0"/>
         <geometry>
-          <mesh filename="${COLLISION_MESH_PATH}/Gripper_v23.2.STL" scale="0.001 0.001 0.001"/>
+          <mesh filename="${COLLISION_MESH_PATH}/R_Link7.stl" scale="1.0 1.0 1.0"/>
         </geometry>
       </collision>
@@ -37,5 +37,5 @@
         <origin rpy="0 0 0" xyz="0.0 0.0 0.0"/>
         <geometry>
-          <mesh filename="${VISUAL_MESH_PATH}/R_GripperA.stl" scale="0.001 0.001 0.001"/>
+          <mesh filename="${VISUAL_MESH_PATH}/R_GripperA.stl" scale="1.0 1.0 1.0"/>
         </geometry>
         <material name="${COLOR_LINK_GRIPPER}"/>
@@ -44,5 +44,5 @@
         <origin rpy="0 0 0" xyz="0.0 0.0 0.0"/>
         <geometry>
-          <mesh filename="${COLLISION_MESH_PATH}/R_GripperA.stl" scale="0.001 0.001 0.001"/>
+          <mesh filename="${COLLISION_MESH_PATH}/R_GripperA.stl" scale="1.0 1.0 1.0"/>
         </geometry>
       </collision>
@@ -57,5 +57,5 @@
         <origin rpy="0 0 3.14" xyz="0.0 0.0 0.0"/>
         <geometry>
-            <mesh filename="${VISUAL_MESH_PATH}/Tong.stl" scale="0.001 0.001 0.001"/>
+            <mesh filename="${VISUAL_MESH_PATH}/Tong.stl" />
         </geometry>
         <material name="${COLOR_LINK_GRIPPER}"/>
@@ -64,5 +64,5 @@
         <origin rpy="0 0 3.14" xyz="0.0 0.0 0.0"/>
         <geometry>
-          <mesh filename="${COLLISION_MESH_PATH}/Tong.stl" scale="0.001 0.001 0.001"/>
+          <mesh filename="${COLLISION_MESH_PATH}/Tong.stl" />
         </geometry>
       </collision>
@@ -97,5 +97,5 @@
         <origin rpy="0 0 0" xyz="0.0 0.0 0.0"/>
         <geometry>
-          <mesh filename="${VISUAL_MESH_PATH}/R_GripperB.stl" scale="0.001 0.001 0.001"/>
+          <mesh filename="${VISUAL_MESH_PATH}/R_GripperB.stl" scale="1.0 1.0 1.0"/>
         </geometry>
         <material name="${COLOR_LINK_GRIPPER}"/>
@@ -104,5 +104,5 @@
         <origin rpy="0 0 0" xyz="0.0 0.0 0.0"/>
         <geometry>
-          <mesh filename="${COLLISION_MESH_PATH}/R_GripperB.stl" scale="0.001 0.001 0.001"/>
+          <mesh filename="${COLLISION_MESH_PATH}/R_GripperB.stl" scale="1.0 1.0 1.0"/>
         </geometry>
       </collision>
@@ -117,5 +117,5 @@
         <origin rpy="0 0 0" xyz="0.0 0.0 0.0"/>
         <geometry>
-            <mesh filename="${VISUAL_MESH_PATH}/Tong.stl" scale="0.001 0.001 0.001"/>
+            <mesh filename="${VISUAL_MESH_PATH}/Tong.stl" />
         </geometry>
         <material name="${COLOR_LINK_GRIPPER}"/>
@@ -124,5 +124,5 @@
         <origin rpy="0 0 0" xyz="0.0 0.0 0.0"/>
         <geometry>
-          <mesh filename="${COLLISION_MESH_PATH}/Tong.stl" scale="0.001 0.001 0.001"/>
+          <mesh filename="${COLLISION_MESH_PATH}/Tong.stl" />
         </geometry>
       </collision>
